File: Wildlife_Cam_PCB/Lapse_O_Matic_PCB.kicad_pcb (KiCad board)
At the start: 2 copper layers, 39.9 x 79.9 mm, 38 parts, among them J1 PIR, J10 POWER, J11 LOGO4, J2 TRIG, J3 RTC_DS3231, J4 PROG, J5 PROG_EN, J6 LOGO1, J7 LOGO2, J8 PCB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

Commit message: PCB updates
Updated PCB
Other:
- rule pad_to_mask_clearance: 0.2 -> 0
