File: Lapse-O-Matic_PCB/Lapse_O_Matic_PCB.sch (KiCad schematic (older format))
At the start: 38 parts, among them J1 PIR, J10 POWER, J11 LOGO4, J2 TRIG, J3 RTC_DS3231, J4 PROG, J5 PROG_EN, J6 LOGO1, J7 LOGO2, J8 PCB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

Commit message: updated PCB and hardware
Parts:
- added J12: PCB_Solar, symbol Connector_Generic:Conn_01x01
- added R3, R4: 1k, REInnovationFootprint:TH_Resistor_1, symbol Device:R
- C1, C3: symbol device:CP -> Device:CP
- D4, D5, D6, D7, D8: symbol WildlifeCamera_PCB-rescue:LED-device -> matts_components:LED
- J1: symbol WildlifeCamera_PCB-rescue:Conn_01x03-Connector_Generic -> Connector_Generic:Conn_01x03
- J2: value TRIG -> TRIGGER; footprint REInnovationFootprint:SIL-3_lg_pad -> REInnovationFootprint:SIL-3_screw_terminal; symbol WildlifeCamera_PCB-rescue:Conn_01x03-Connector_Generic -> Connector_Generic:Conn_01x03
- J4: symbol WildlifeCamera_PCB-rescue:Conn_01x06-Connector_Generic -> Connector_Generic:Conn_01x06
- J5: symbol WildlifeCamera_PCB-rescue:Conn_01x02-Connector_Generic -> Connector_Generic:Conn_01x02
- J8: footprint REInnovationFootprint:PCB_SolarChargerPCB40x80 -> REInnovationFootprint:PCB_Lapse-O-Matic
- J9: footprint REInnovationGraphics:lapseomatic logo -> REInnovationGraphics:lapseomatic logo_20x6mm
- Q3: symbol WildlifeCamera_PCB-rescue:Q_NPN_BCE-Device -> Device:Q_NPN_BCE
- R1, R10, R11, R12, R13, R14, R15, R16, R2, R6, R8, R9: symbol WildlifeCamera_PCB-rescue:R-Device -> Device:R
- SW2: symbol WildlifeCamera_PCB-rescue:SW_Push-Switch -> matts_components:SW_PUSH
Connections:
- net U0R: now also R3.2; no longer J4.4 (Pin_4)
- net U0T: now also R4.2; no longer J4.5 (Pin_5)
- new net: J4.4 (Pin_4), R3.1
- new net: J4.5 (Pin_5), R4.1
- no-connect marks 12 -> 13
Other:
- moved on the sheet: C1, C3, J10, J4, J5, Q3, R10, R11, R12, R13, R14, R15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
